Commit message: part 2 working

File: urdf/macros.xacro (robot description, xacro)
@@ -1,4 +1,4 @@
 <?xml version="1.0"?>
-<robot>
+<robot xmlns:xacro="http://www.ros.org/wiki/xacro">
   <macro name="cylinder_inertial" params="name m r h">
     <inertial name="${name}_intertial">
@@ -25,3 +25,25 @@
     </inertial>
   </macro>
+  <macro name="wheel" params="id m r w x y z">
+    <joint name="wheel_joint_${id}" type="continuous">
+      <axis xyz="0 1 0" />
+      <origin xyz="${x} ${y} ${z}" rpy="0 0 0"/>
+      <parent link="chassis"/>
+      <child link="wheel_${id}"/>
+    </joint>
+    <link name='wheel_${id}'>
+      <xacro:cylinder_inertial name="wheel_${id}_inertial" m="${m}" r="${r}" h="${w}"/>
+      <collision name='wheel_${id}_collision'>
+        <geometry>
+          <cylinder radius="${r}" length="${w}"/>
+        </geometry>
+      </collision>
+      <visual name='wheel_${id}_visual'>
+        <origin xyz="0 0 0" rpy="${pi / 2} 0 0"/>
+        <geometry>
+          <cylinder radius="${r}" length="${w}"/>
+        </geometry>
+      </visual>
+    </link>
+  </macro>
 </robot>

File: urdf/robot.xacro (robot description, xacro)
@@ -3,9 +3,15 @@
   <xacro:property name="chassis_width" value="0.15"/>
   <xacro:property name="chassis_length" value="0.2"/>
-  <xacro:property name="chassis_height" value="0.05"/>
+  <xacro:property name="chassis_height" value="0.06"/>
   <xacro:property name="chassis_mass" value="0.5"/>
+  <xacro:property name="chassis_z_offset" value="0.02"/>
   <xacro:property name="wheel_radius" value="0.04"/>
-  <xacro:property name="wheel_width" value="0.03"/>
-  <xacro:include filename="$(find enph353_ros_lab)/urdf/robot.gazebo" />
+  <xacro:property name="wheel_width" value="0.01"/>
+  <xacro:property name="wheel_offset" value="0.03"/>
+  <xacro:property name="wheel_mass" value="0.04"/>
+   <xacro:property name="wheel_z_offset" value="${wheel_radius - 0.5 * chassis_height}"/>
+  <xacro:property name="camera_link" value="0.05" /> <!-- Size of square 'camera' box -->
+  <xacro:property name="camera_z_offset" value="0.0" />
+  <!-- <xacro:include filename="$(find enph353_ros_lab)/urdf/robot.gazebo" /> -->
   <xacro:include filename="$(find enph353_ros_lab)/urdf/macros.xacro" />
   <link name='chassis'>
@@ -17,5 +23,5 @@
     </collision>
     <visual name='chassis_visual'>
-      <origin xyz="0 0 0" rpy=" 0 0 0"/>
+      <origin xyz="0 0 ${chassis_z_offset}" rpy=" 0 0 0"/>
       <geometry>
         <box size="${chassis_length} ${chassis_width} ${chassis_height}"/>
@@ -23,3 +29,96 @@
     </visual>
   </link>
+  <joint name="camera_joint" type="fixed">
+    <axis xyz="1 0 -1" />
+    <origin xyz="${chassis_length * 0.5 - camera_link * 0.5} 0 ${chassis_height * 0.5 + camera_link * 0.5}" rpy="0 0 0"/>
+    <parent link="chassis"/>
+    <child link="camera_link"/>
+  </joint>
+  <!-- Camera -->
+  <link name="camera_link">
+    <collision>
+      <origin xyz="0 0 0" rpy="0 0 0"/>
+      <geometry>
+    <box size="${camera_link} ${camera_link} ${camera_link}"/>
+      </geometry>
+    </collision>
+    <visual>
+      <origin xyz="0 0 0" rpy="0 0 0"/>
+      <geometry>
+    <box size="${camera_link} ${camera_link} ${camera_link}"/>
+      </geometry>
+      <material name="red"/>
+    </visual>
+    <inertial>
+      <mass value="1e-5" />
+      <origin xyz="0 0 0" rpy="0 0 0"/>
+      <inertia ixx="1e-6" ixy="0" ixz="0" iyy="1e-6" iyz="0" izz="1e-6" />
+    </inertial>
+  </link>
+  <!-- 1: top-left, 2: top-right, 3: bottom-left, 4: bottom-right -->
+  <wheel id="1" m="${wheel_mass}" r="${wheel_radius}" w="${wheel_width}"
+    x="${chassis_length * 0.5 - wheel_offset}" y="${chassis_width * 0.5 + wheel_width * 0.5}" z="${wheel_z_offset}"/>
+  <wheel id="2" m="${wheel_mass}" r="${wheel_radius}" w="${wheel_width}"
+    x="${chassis_length * 0.5 - wheel_offset}" y="${-chassis_width * 0.5 - wheel_width * 0.5}" z="${wheel_z_offset}"/>
+  <wheel id="3" m="${wheel_mass}" r="${wheel_radius}" w="${wheel_width}"
+    x="${-chassis_length* 0.5 + wheel_offset}" y="${chassis_width * 0.5 + wheel_width * 0.5}" z="${wheel_z_offset}"/>
+  <wheel id="4" m="${wheel_mass}" r="${wheel_radius}" w="${wheel_width}"
+    x="${-chassis_length * 0.5 + wheel_offset}" y="${-chassis_width * 0.5 - wheel_width * 0.5}" z="${wheel_z_offset}"/>
+  <!-- camera -->
+  <gazebo reference="camera_link">
+    <sensor type="camera" name="camera1">
+      <update_rate>30.0</update_rate>
+      <camera name="head">
+        <horizontal_fov>1.3962634</horizontal_fov>
+        <image>
+          <width>800</width>
+          <height>800</height>
+          <format>R8G8B8</format>
+        </image>
+        <clip>
+          <near>0.02</near>
+          <far>300</far>
+        </clip>
+        <noise>
+          <type>gaussian</type>
+          <!-- Noise is sampled independently per pixel on each frame.
+               That pixel's noise value is added to each of its color
+               channels, which at that point lie in the range [0,1]. -->
+          <mean>0.0</mean>
+          <stddev>0.007</stddev>
+        </noise>
+      </camera>
+      <plugin name="camera_controller" filename="libgazebo_ros_camera.so">
+        <alwaysOn>true</alwaysOn>
+        <updateRate>0.0</updateRate>
+        <cameraName>robot/camera1</cameraName>
+        <imageTopicName>image_raw</imageTopicName>
+        <cameraInfoTopicName>camera_info</cameraInfoTopicName>
+        <frameName>camera_link</frameName>
+        <hackBaseline>0.07</hackBaseline>
+        <distortionK1>0.0</distortionK1>
+        <distortionK2>0.0</distortionK2>
+        <distortionK3>0.0</distortionK3>
+        <distortionT1>0.0</distortionT1>
+        <distortionT2>0.0</distortionT2>
+      </plugin>
+    </sensor>
+  </gazebo>
+  <gazebo>
+    <plugin name="differential_drive_controller" filename="libgazebo_ros_diff_drive.so">
+      <alwaysOn>true</alwaysOn>
+      <updateRate>30.0</updateRate>
+      <leftJoint>wheel_joint_3</leftJoint>
+      <rightJoint>wheel_joint_4</rightJoint>
+      <wheelSeparation>${chassis_width + wheel_width}</wheelSeparation>
+      <wheelDiameter>${wheel_radius * 0.5}</wheelDiameter>
+      <!-- <wheelSeparation>0.16</wheelSeparation>
+      <wheelDiameter>0.08</wheelDiameter> -->
+      <torque>20</torque>
+      <commandTopic>cmd_vel</commandTopic>
+      <odometryTopic>odom</odometryTopic>
+      <odometryFrame>odom</odometryFrame>
+      <robotBaseFrame>base_footprint</robotBaseFrame>
+    </plugin>
+  </gazebo>
 </robot>
